Commit message: feat(urdf): update urdf

File: urdf/komarm.urdf (robot description, URDF)
Before this commit: robot arm_main, 6 links, 5 joints
Links:
- removed link base_mount_v2_1
- removed link hand_rotation_v13_4
- removed link hand_v17_1
- removed link servo_holder2_v9_1
- removed link servo_holder_v23_3
- added link DZ47B-63_circuit_breaker_holder_v3_1, mass 0.012274791356152887; collision mesh filename=../meshes/DZ47B-63_circuit_breaker_holder_v3_1.stl scale=0.001 0.001 0.001; visual mesh filename=../meshes/DZ47B-63_circuit_breaker_holder_v3_1.stl scale=0.001 0.001 0.001
- added link arm_bracket_temp_v12_1, mass 0.16496925038992882; collision mesh filename=../meshes/arm_bracket_temp_v12_1.stl scale=0.001 0.001 0.001; visual mesh filename=../meshes/arm_bracket_temp_v12_1.stl scale=0.001 0.001 0.001
- added link arm_root_v1_1, mass 0.3893898243402566; collision mesh filename=../meshes/arm_root_v1_1.stl scale=0.001 0.001 0.001; visual mesh filename=../meshes/arm_root_v1_1.stl scale=0.001 0.001 0.001
- added link hand_finger_v2_1, mass 0.18316176934492862; collision mesh filename=../meshes/hand_finger_v2_1.stl scale=0.001 0.001 0.001; visual mesh filename=../meshes/hand_finger_v2_1.stl scale=0.001 0.001 0.001
- added link hand_unit_v1_1, mass 0.6163609537224307; collision mesh filename=../meshes/hand_unit_v1_1.stl scale=0.001 0.001 0.001; visual mesh filename=../meshes/hand_unit_v1_1.stl scale=0.001 0.001 0.001
- added link lipo_bracket_v5_1, mass 0.15095338739595293; collision mesh filename=../meshes/lipo_bracket_v5_1.stl scale=0.001 0.001 0.001; visual mesh filename=../meshes/lipo_bracket_v5_1.stl scale=0.001 0.001 0.001
- added link pitch_1_test_v1_1, mass 0.5173712582672985; collision mesh filename=../meshes/pitch_1_test_v1_1.stl scale=0.001 0.001 0.001; visual mesh filename=../meshes/pitch_1_test_v1_1.stl scale=0.001 0.001 0.001
- added link pitch_2_test_v1_1, mass 0.4049688490988578; collision mesh filename=../meshes/pitch_2_test_v1_1.stl scale=0.001 0.001 0.001; visual mesh filename=../meshes/pitch_2_test_v1_1.stl scale=0.001 0.001 0.001
- added link raspi4_bracket_v1_1, mass 0.10292684148685698; collision mesh filename=../meshes/raspi4_bracket_v1_1.stl scale=0.001 0.001 0.001; visual mesh filename=../meshes/raspi4_bracket_v1_1.stl scale=0.001 0.001 0.001
- added link raspi4_v2_1, mass 0.7390104624417327; collision mesh filename=../meshes/raspi4_v2_1.stl scale=0.001 0.001 0.001; visual mesh filename=../meshes/raspi4_v2_1.stl scale=0.001 0.001 0.001
- added link roll_1_test_v1_1, mass 0.45569427768407117; collision mesh filename=../meshes/roll_1_test_v1_1.stl scale=0.001 0.001 0.001; visual mesh filename=../meshes/roll_1_test_v1_1.stl scale=0.001 0.001 0.001
- added link roll_2_test_v1_1, mass 0.45660397486942944; collision mesh filename=../meshes/roll_2_test_v1_1.stl scale=0.001 0.001 0.001; visual mesh filename=../meshes/roll_2_test_v1_1.stl scale=0.001 0.001 0.001
- added link wheel_control_board_v7_1, mass 0.05597515361092653; collision mesh filename=../meshes/wheel_control_board_v7_1.stl scale=0.001 0.001 0.001; visual mesh filename=../meshes/wheel_control_board_v7_1.stl scale=0.001 0.001 0.001
- added link wheel_control_board_v7_2, mass 0.05597515361092653; collision mesh filename=../meshes/wheel_control_board_v7_2.stl scale=0.001 0.001 0.001; visual mesh filename=../meshes/wheel_control_board_v7_2.stl scale=0.001 0.001 0.001
- link base_link: mass 0.3900830776668987 -> 4.116732793254999
Joints:
- removed joint Revolute 11
- removed joint Revolute 12
- removed joint Revolute 7
- removed joint Revolute 8
- removed joint Revolute 9
- added joint Revolute 1: type revolute, parent arm_root_v1_1, child pitch_1_test_v1_1, origin xyz=0.03568 -0.0206 0.01305 rpy=0 0 0, axis -0.0 0.0 -1.0, limit lower=-1.570796 upper=1.570796 effort=100 velocity=100
- added joint Revolute_2: type revolute, parent pitch_1_test_v1_1, child roll_1_test_v1_1, origin xyz=0.043692 -0.048724 0.00545 rpy=0 0 0, axis 0.5 0.866025 -0.0, limit lower=-1.396263 upper=1.919862 effort=100 velocity=100
- added joint Revolute_3: type continuous, parent roll_1_test_v1_1, child pitch_2_test_v1_1, origin xyz=0.059443 -0.00984 0.0 rpy=0 0 0, axis 0.866025 -0.5 0.0
- added joint Revolute_4: type revolute, parent pitch_2_test_v1_1, child roll_2_test_v1_1, origin xyz=0.029511 -0.041287 0.0 rpy=0 0 0, axis 0.5 0.866025 0.0, limit lower=-1.48353 upper=1.919862 effort=100 velocity=100
- added joint Revolute_5: type continuous, parent roll_2_test_v1_1, child hand_unit_v1_1, origin xyz=0.059444 -0.00984 0.0 rpy=0 0 0, axis -0.866025 0.5 -0.0
- added joint Revolute_6: type revolute, parent hand_unit_v1_1, child hand_finger_v2_1, origin xyz=0.011113 -0.032051 0.013 rpy=0 0 0, axis 0.5 0.866025 0.0, limit lower=-1.047198 upper=0.872665 effort=100 velocity=100
- added joint Rigid 16: type fixed, parent base_link, child lipo_bracket_v5_1, origin xyz=-0.040468 0.155581 0.0365 rpy=0 0 0
- added joint Rigid 17: type fixed, parent base_link, child DZ47B-63_circuit_breaker_holder_v3_1, origin xyz=-0.088434 0.095997 0.0365 rpy=0 0 0
- added joint Rigid 26: type fixed, parent arm_bracket_temp_v12_1, child arm_root_v1_1, origin xyz=0.017558 0.001411 0.04 rpy=0 0 0
- added joint Rigid 27: type fixed, parent base_link, child wheel_control_board_v7_1, origin xyz=-0.03065 0.04435 0.0365 rpy=0 0 0
- added joint Rigid 4: type fixed, parent base_link, child arm_bracket_temp_v12_1, origin xyz=0.035703 0.064664 0.0365 rpy=0 0 0
- added joint Rigid 6: type fixed, parent wheel_control_board_v7_1, child wheel_control_board_v7_2, origin xyz=0.018859 0.077391 0.0016 rpy=0 0 0
- added joint Rigid 7: type fixed, parent base_link, child raspi4_bracket_v1_1, origin xyz=0.0 0.176825 0.0365 rpy=0 0 0
- added joint Rigid 8: type fixed, parent raspi4_bracket_v1_1, child raspi4_v2_1, origin xyz=0.0 -0.013 0.021 rpy=0 0 0

File: urdf/materials.xacro (robot description, xacro)
@@ -1,4 +1,4 @@
 <?xml version="1.0" ?>
-<robot name="arm_main" xmlns:xacro="http://www.ros.org/wiki/xacro" >
+<robot name="assembly_main" xmlns:xacro="http://www.ros.org/wiki/xacro" >
 <material name="silver_default">
   <color rgba="0.700 0.700 0.700 1.000"/>
@@ -7,3 +7,6 @@
   <color rgba="0.6274509803921569 0.6274509803921569 0.6274509803921569 1.0"/>
 </material>
+<material name="aluminum_satin">
+  <color rgba="0.9607843137254902 0.9607843137254902 0.9647058823529412 1.0"/>
+</material>
 </robot>

Commit message: feat(koma): add value

File: urdf/komarm.urdf (robot description, URDF)
Before this commit: robot assembly_main, 13 links, 12 joints
Links:
- link base_link: mass 4.116732793254999 -> 20.0

Commit message: fix(urdf): joint name

File: urdf/komarm.urdf (robot description, URDF)
Before this commit: robot assembly_main, 13 links, 12 joints
Joints:
- removed joint Revolute 1
- added joint Revolute_1: type revolute, parent arm_root_v1_1, child pitch_1_test_v1_1, origin xyz=0.03568 -0.0206 0.01305 rpy=0 0 0, axis -0.0 0.0 -1.0, limit lower=-1.570796 upper=1.570796 effort=100 velocity=100

Commit message: fix(urdf): revolute 1

File: urdf/komarm.urdf (robot description, URDF)
Before this commit: robot assembly_main, 13 links, 12 joints
Joints:
- removed joint Revolute 1
- added joint Revolute_1: type revolute, parent arm_root_v4_1, child pitch_1_test_v3_1, origin xyz=0.03568 -0.0206 0.01305 rpy=0 0 0, axis -0.0 0.0 -1.0, limit lower=-1.570796 upper=1.570796 effort=100 velocity=100

Commit message: feat(limit): add vel and effort limit

File: urdf/komarm.urdf (robot description, URDF)
Before this commit: robot assembly_main, 13 links, 12 joints
Joints:
- joint Revolute_1: limit lower=-1.570796 upper=1.570796 effort=100 velocity=100 -> lower=-1.570796 upper=1.570796 effort=1.5 velocity=4.0
- joint Revolute_2: limit lower=-1.396263 upper=1.919862 effort=100 velocity=100 -> lower=-1.396263 upper=1.919862 effort=1.5 velocity=4.0
- joint Revolute_3: limit (none) -> effort=1.5 velocity=4.0
- joint Revolute_4: limit lower=-1.48353 upper=1.919862 effort=100 velocity=100 -> lower=-1.48353 upper=1.919862 effort=1.5 velocity=4.0
- joint Revolute_5: limit (none) -> effort=1.5 velocity=4.0
- joint Revolute_6: limit lower=-1.047198 upper=0.872665 effort=100 velocity=100 -> lower=-1.047198 upper=0.872665 effort=1.5 velocity=4.0

Commit message: feat(collision): delete arm collision

File: urdf/komarm.urdf (robot description, URDF)
Before this commit: robot assembly_main, 13 links, 12 joints
Links:
- link arm_root_v4_1: geometry visual mesh filename=../meshes/arm_root_v4_1.stl scale=0.001 0.001 0.001
- link hand_finger_v7_1: geometry visual mesh filename=../meshes/hand_finger_v7_1.stl scale=0.001 0.001 0.001
- link hand_unit_v3_1: geometry visual mesh filename=../meshes/hand_unit_v3_1.stl scale=0.001 0.001 0.001
- link pitch_1_test_v3_1: geometry visual mesh filename=../meshes/pitch_1_test_v3_1.stl scale=0.001 0.001 0.001
- link pitch_2_test_v3_1: geometry visual mesh filename=../meshes/pitch_2_test_v3_1.stl scale=0.001 0.001 0.001
- link roll_1_test_v3_1: geometry visual mesh filename=../meshes/roll_1_test_v3_1.stl scale=0.001 0.001 0.001
- link roll_2_test_v3_1: geometry visual mesh filename=../meshes/roll_2_test_v3_1.stl scale=0.001 0.001 0.001

Commit message: fix(launch): weight

File: urdf/komarm.urdf (robot description, URDF)
Before this commit: robot assembly_main, 16 links, 15 joints
Links:
- link base_link: mass 4.27590428722208 -> 10.0
