Commit message: fix(name): - to _

File: urdf/assembly_main.xacro (robot description, xacro)
@@ -43,24 +43,4 @@
   </collision>
 </link>
-<link name="wheel_control_board_v7_2">
-  <inertial>
-    <origin xyz="-0.008950875512003416 -0.039393966482722906 0.10000262508964408" rpy="0 0 0"/>
-    <mass value="0.05597515361092653"/>
-    <inertia ixx="2.1e-05" iyy="1.9e-05" izz="4e-05" ixy="-1e-05" iyz="0.0" ixz="-0.0"/>
-  </inertial>
-  <visual>
-    <origin xyz="0.011791 -0.121741 -0.0381" rpy="0 0 0"/>
-    <geometry>
-      <mesh filename="package://assembly_main_description/meshes/wheel_control_board_v7_2.stl" scale="0.001 0.001 0.001"/>
-    </geometry>
-    <material name="steel_satin"/>
-  </visual>
-  <collision>
-    <origin xyz="0.011791 -0.121741 -0.0381" rpy="0 0 0"/>
-    <geometry>
-      <mesh filename="package://assembly_main_description/meshes/wheel_control_board_v7_2.stl" scale="0.001 0.001 0.001"/>
-    </geometry>
-  </collision>
-</link>
 <link name="raspi4_bracket_v1_1">
   <inertial>
@@ -123,5 +103,5 @@
   </collision>
 </link>
-<link name="DZ47B-63_circuit_breaker_holder_v3_1">
+<link name="DZ47B_63_circuit_breaker_holder_v3_1">
   <inertial>
     <origin xyz="0.02229875370121319 -0.03862280991922731 0.002938007686629586" rpy="0 0 0"/>
@@ -132,5 +112,5 @@
     <origin xyz="0.088434 -0.095997 -0.0365" rpy="0 0 0"/>
     <geometry>
-      <mesh filename="package://assembly_main_description/meshes/DZ47B-63_circuit_breaker_holder_v3_1.stl" scale="0.001 0.001 0.001"/>
+      <mesh filename="package://assembly_main_description/meshes/DZ47B_63_circuit_breaker_holder_v3_1.stl" scale="0.001 0.001 0.001"/>
     </geometry>
     <material name="steel_satin"/>
@@ -139,5 +119,5 @@
     <origin xyz="0.088434 -0.095997 -0.0365" rpy="0 0 0"/>
     <geometry>
-      <mesh filename="package://assembly_main_description/meshes/DZ47B-63_circuit_breaker_holder_v3_1.stl" scale="0.001 0.001 0.001"/>
+      <mesh filename="package://assembly_main_description/meshes/DZ47B_63_circuit_breaker_holder_v3_1.stl" scale="0.001 0.001 0.001"/>
     </geometry>
   </collision>
@@ -160,24 +140,4 @@
     <geometry>
       <mesh filename="package://assembly_main_description/meshes/arm_root_v1_1.stl" scale="0.001 0.001 0.001"/>
-    </geometry>
-  </collision>
-</link>
-<link name="wheel_control_board_v7_1">
-  <inertial>
-    <origin xyz="0.009908124487998424 0.03799703351727894 0.0016026250896445035" rpy="0 0 0"/>
-    <mass value="0.05597515361092653"/>
-    <inertia ixx="2.1e-05" iyy="1.9e-05" izz="4e-05" ixy="-1e-05" iyz="0.0" ixz="-0.0"/>
-  </inertial>
-  <visual>
-    <origin xyz="0.03065 -0.04435 -0.0365" rpy="0 0 0"/>
-    <geometry>
-      <mesh filename="package://assembly_main_description/meshes/wheel_control_board_v7_1.stl" scale="0.001 0.001 0.001"/>
-    </geometry>
-    <material name="steel_satin"/>
-  </visual>
-  <collision>
-    <origin xyz="0.03065 -0.04435 -0.0365" rpy="0 0 0"/>
-    <geometry>
-      <mesh filename="package://assembly_main_description/meshes/wheel_control_board_v7_1.stl" scale="0.001 0.001 0.001"/>
     </geometry>
   </collision>
@@ -308,9 +268,4 @@
   <child link="arm_bracket_temp_v12_1"/>
 </joint>
-<joint name="Rigid 6" type="fixed">
-  <origin xyz="0.018859 0.077391 0.0016" rpy="0 0 0"/>
-  <parent link="wheel_control_board_v7_1"/>
-  <child link="wheel_control_board_v7_2"/>
-</joint>
 <joint name="Rigid 7" type="fixed">
   <origin xyz="0.0 0.176825 0.0365" rpy="0 0 0"/>
@@ -331,5 +286,5 @@
   <origin xyz="-0.088434 0.095997 0.0365" rpy="0 0 0"/>
   <parent link="base_link"/>
-  <child link="DZ47B-63_circuit_breaker_holder_v3_1"/>
+  <child link="DZ47B_63_circuit_breaker_holder_v3_1"/>
 </joint>
 <joint name="Rigid 26" type="fixed">
@@ -337,9 +292,4 @@
   <parent link="arm_bracket_temp_v12_1"/>
   <child link="arm_root_v1_1"/>
-</joint>
-<joint name="Rigid 27" type="fixed">
-  <origin xyz="-0.03065 0.04435 0.0365" rpy="0 0 0"/>
-  <parent link="base_link"/>
-  <child link="wheel_control_board_v7_1"/>
 </joint>
 <joint name="Revolute 1" type="revolute">

File: urdf/komarm.urdf (robot description, URDF)
Before this commit: robot assembly_main, 15 links, 14 joints
Links:
- removed link DZ47B-63_circuit_breaker_holder_v3_1
- removed link wheel_control_board_v7_1
- removed link wheel_control_board_v7_2
- added link DZ47B_63_circuit_breaker_holder_v3_1, mass 0.012274791356152887; collision mesh filename=../meshes/DZ47B_63_circuit_breaker_holder_v3_1.stl scale=0.001 0.001 0.001; visual mesh filename=../meshes/DZ47B_63_circuit_breaker_holder_v3_1.stl scale=0.001 0.001 0.001
Joints:
- removed joint Rigid 27
- removed joint Rigid 6
- joint Rigid 17: child DZ47B-63_circuit_breaker_holder_v3_1 -> DZ47B_63_circuit_breaker_holder_v3_1

Commit message: fix(launch): weight

File: urdf/assembly_main.xacro (robot description, xacro)
@@ -123,141 +123,141 @@
   </collision>
 </link>
-<link name="arm_root_v1_1">
-  <inertial>
-    <origin xyz="0.019613622126277777 -0.011324599028677579 -0.009707737296854035" rpy="0 0 0"/>
-    <mass value="0.3893898243402566"/>
-    <inertia ixx="8.6e-05" iyy="0.000116" izz="0.000111" ixy="2.6e-05" iyz="1e-06" ixz="-1e-06"/>
+<link name="arm_root_v4_1">
+  <inertial>
+    <origin xyz="0.022163724443126365 -0.012796901291084212 -0.009138901606431687" rpy="0 0 0"/>
+    <mass value="0.06457976620923557"/>
+    <inertia ixx="1.6e-05" iyy="2.1e-05" izz="1.9e-05" ixy="5e-06" iyz="0.0" ixz="-1e-06"/>
   </inertial>
   <visual>
     <origin xyz="-0.053261 -0.066075 -0.0765" rpy="0 0 0"/>
     <geometry>
-      <mesh filename="package://assembly_main_description/meshes/arm_root_v1_1.stl" scale="0.001 0.001 0.001"/>
-    </geometry>
-    <material name="steel_satin"/>
+      <mesh filename="package://assembly_main_description/meshes/arm_root_v4_1.stl" scale="0.001 0.001 0.001"/>
+    </geometry>
+    <material name="abs_white"/>
   </visual>
   <collision>
     <origin xyz="-0.053261 -0.066075 -0.0765" rpy="0 0 0"/>
     <geometry>
-      <mesh filename="package://assembly_main_description/meshes/arm_root_v1_1.stl" scale="0.001 0.001 0.001"/>
-    </geometry>
-  </collision>
-</link>
-<link name="pitch_1_test_v1_1">
-  <inertial>
-    <origin xyz="0.0328465922924564 -0.018706756231211926 -0.0010892901314617925" rpy="0 0 0"/>
-    <mass value="0.5173712582672985"/>
-    <inertia ixx="0.000196" iyy="0.000247" izz="0.000212" ixy="3.9e-05" iyz="3.1e-05" ixz="-5.5e-05"/>
+      <mesh filename="package://assembly_main_description/meshes/arm_root_v4_1.stl" scale="0.001 0.001 0.001"/>
+    </geometry>
+  </collision>
+</link>
+<link name="pitch_1_test_v3_1">
+  <inertial>
+    <origin xyz="0.0358303038564968 -0.019899545668259706 -0.00013072073296151177" rpy="0 0 0"/>
+    <mass value="0.08186133563123103"/>
+    <inertia ixx="3e-05" iyy="4e-05" izz="3.7e-05" ixy="6e-06" iyz="5e-06" ixz="-9e-06"/>
   </inertial>
   <visual>
     <origin xyz="-0.088941 -0.045475 -0.08955" rpy="0 0 0"/>
     <geometry>
-      <mesh filename="package://assembly_main_description/meshes/pitch_1_test_v1_1.stl" scale="0.001 0.001 0.001"/>
-    </geometry>
-    <material name="steel_satin"/>
+      <mesh filename="package://assembly_main_description/meshes/pitch_1_test_v3_1.stl" scale="0.001 0.001 0.001"/>
+    </geometry>
+    <material name="abs_white"/>
   </visual>
   <collision>
     <origin xyz="-0.088941 -0.045475 -0.08955" rpy="0 0 0"/>
     <geometry>
-      <mesh filename="package://assembly_main_description/meshes/pitch_1_test_v1_1.stl" scale="0.001 0.001 0.001"/>
-    </geometry>
-  </collision>
-</link>
-<link name="roll_1_test_v1_1">
-  <inertial>
-    <origin xyz="0.04136948087302786 0.0005946999542336038 0.017590075270092265" rpy="0 0 0"/>
-    <mass value="0.45569427768407117"/>
-    <inertia ixx="0.000154" iyy="0.000161" izz="0.00013" ixy="6e-06" iyz="5e-06" ixz="-9e-06"/>
+      <mesh filename="package://assembly_main_description/meshes/pitch_1_test_v3_1.stl" scale="0.001 0.001 0.001"/>
+    </geometry>
+  </collision>
+</link>
+<link name="roll_1_test_v3_1">
+  <inertial>
+    <origin xyz="0.042100640863960814 0.00017256453450652937 0.015160914691842262" rpy="0 0 0"/>
+    <mass value="0.07353297901744495"/>
+    <inertia ixx="2.5e-05" iyy="2.7e-05" izz="2.1e-05" ixy="2e-06" iyz="0.0" ixz="-0.0"/>
   </inertial>
   <visual>
     <origin xyz="-0.132633 0.003249 -0.095" rpy="0 0 0"/>
     <geometry>
-      <mesh filename="package://assembly_main_description/meshes/roll_1_test_v1_1.stl" scale="0.001 0.001 0.001"/>
-    </geometry>
-    <material name="steel_satin"/>
+      <mesh filename="package://assembly_main_description/meshes/roll_1_test_v3_1.stl" scale="0.001 0.001 0.001"/>
+    </geometry>
+    <material name="abs_white"/>
   </visual>
   <collision>
     <origin xyz="-0.132633 0.003249 -0.095" rpy="0 0 0"/>
     <geometry>
-      <mesh filename="package://assembly_main_description/meshes/roll_1_test_v1_1.stl" scale="0.001 0.001 0.001"/>
-    </geometry>
-  </collision>
-</link>
-<link name="pitch_2_test_v1_1">
-  <inertial>
-    <origin xyz="0.02310996157289455 -0.013751811536932397 -2.9731213324613037e-10" rpy="0 0 0"/>
-    <mass value="0.4049688490988578"/>
-    <inertia ixx="8.5e-05" iyy="0.000109" izz="0.000143" ixy="1.7e-05" iyz="0.0" ixz="-0.0"/>
+      <mesh filename="package://assembly_main_description/meshes/roll_1_test_v3_1.stl" scale="0.001 0.001 0.001"/>
+    </geometry>
+  </collision>
+</link>
+<link name="pitch_2_test_v3_1">
+  <inertial>
+    <origin xyz="0.025973068908376362 -0.014769408547619371 -2.946918264967735e-10" rpy="0 0 0"/>
+    <mass value="0.06668343069893205"/>
+    <inertia ixx="1.5e-05" iyy="1.9e-05" izz="2.6e-05" ixy="2e-06" iyz="0.0" ixz="-0.0"/>
   </inertial>
   <visual>
     <origin xyz="-0.192076 0.013089 -0.095" rpy="0 0 0"/>
     <geometry>
-      <mesh filename="package://assembly_main_description/meshes/pitch_2_test_v1_1.stl" scale="0.001 0.001 0.001"/>
-    </geometry>
-    <material name="steel_satin"/>
+      <mesh filename="package://assembly_main_description/meshes/pitch_2_test_v3_1.stl" scale="0.001 0.001 0.001"/>
+    </geometry>
+    <material name="abs_white"/>
   </visual>
   <collision>
     <origin xyz="-0.192076 0.013089 -0.095" rpy="0 0 0"/>
     <geometry>
-      <mesh filename="package://assembly_main_description/meshes/pitch_2_test_v1_1.stl" scale="0.001 0.001 0.001"/>
-    </geometry>
-  </collision>
-</link>
-<link name="roll_2_test_v1_1">
-  <inertial>
-    <origin xyz="0.041372396148530305 0.0005933410812946349 0.01761719047417358" rpy="0 0 0"/>
-    <mass value="0.45660397486942944"/>
-    <inertia ixx="0.000154" iyy="0.000161" izz="0.00013" ixy="6e-06" iyz="5e-06" ixz="-9e-06"/>
+      <mesh filename="package://assembly_main_description/meshes/pitch_2_test_v3_1.stl" scale="0.001 0.001 0.001"/>
+    </geometry>
+  </collision>
+</link>
+<link name="roll_2_test_v3_1">
+  <inertial>
+    <origin xyz="0.04210189544568463 0.000172164463575597 0.015187663571532464" rpy="0 0 0"/>
+    <mass value="0.07365581710871624"/>
+    <inertia ixx="2.5e-05" iyy="2.7e-05" izz="2.1e-05" ixy="2e-06" iyz="0.0" ixz="-0.0"/>
   </inertial>
   <visual>
     <origin xyz="-0.221587 0.054376 -0.095" rpy="0 0 0"/>
     <geometry>
-      <mesh filename="package://assembly_main_description/meshes/roll_2_test_v1_1.stl" scale="0.001 0.001 0.001"/>
-    </geometry>
-    <material name="steel_satin"/>
+      <mesh filename="package://assembly_main_description/meshes/roll_2_test_v3_1.stl" scale="0.001 0.001 0.001"/>
+    </geometry>
+    <material name="abs_white"/>
   </visual>
   <collision>
     <origin xyz="-0.221587 0.054376 -0.095" rpy="0 0 0"/>
     <geometry>
-      <mesh filename="package://assembly_main_description/meshes/roll_2_test_v1_1.stl" scale="0.001 0.001 0.001"/>
-    </geometry>
-  </collision>
-</link>
-<link name="hand_unit_v1_1">
-  <inertial>
-    <origin xyz="0.02827117996488704 -0.01613952894578953 -0.014188170173815906" rpy="0 0 0"/>
-    <mass value="0.6163609537224307"/>
-    <inertia ixx="0.000331" iyy="0.000439" izz="0.000371" ixy="9.2e-05" iyz="-6e-05" ixz="0.00011"/>
+      <mesh filename="package://assembly_main_description/meshes/roll_2_test_v3_1.stl" scale="0.001 0.001 0.001"/>
+    </geometry>
+  </collision>
+</link>
+<link name="hand_unit_v3_1">
+  <inertial>
+    <origin xyz="0.027318565725242272 -0.01604965279786605 -0.011102966860764008" rpy="0 0 0"/>
+    <mass value="0.0952280970557457"/>
+    <inertia ixx="5.4e-05" iyy="6.8e-05" izz="5.4e-05" ixy="1.1e-05" iyz="-8e-06" ixz="1.7e-05"/>
   </inertial>
   <visual>
     <origin xyz="-0.281031 0.064216 -0.095" rpy="0 0 0"/>
     <geometry>
-      <mesh filename="package://assembly_main_description/meshes/hand_unit_v1_1.stl" scale="0.001 0.001 0.001"/>
-    </geometry>
-    <material name="steel_satin"/>
+      <mesh filename="package://assembly_main_description/meshes/hand_unit_v3_1.stl" scale="0.001 0.001 0.001"/>
+    </geometry>
+    <material name="abs_white"/>
   </visual>
   <collision>
     <origin xyz="-0.281031 0.064216 -0.095" rpy="0 0 0"/>
     <geometry>
-      <mesh filename="package://assembly_main_description/meshes/hand_unit_v1_1.stl" scale="0.001 0.001 0.001"/>
-    </geometry>
-  </collision>
-</link>
-<link name="hand_finger_v2_1">
-  <inertial>
-    <origin xyz="0.042291236138162824 0.0006403953404404278 0.02461729439488529" rpy="0 0 0"/>
-    <mass value="0.18316176934492862"/>
-    <inertia ixx="6.5e-05" iyy="9.8e-05" izz="0.000134" ixy="2.8e-05" iyz="1.3e-05" ixz="-2.3e-05"/>
+      <mesh filename="package://assembly_main_description/meshes/hand_unit_v3_1.stl" scale="0.001 0.001 0.001"/>
+    </geometry>
+  </collision>
+</link>
+<link name="hand_finger_v6_1">
+  <inertial>
+    <origin xyz="0.04229123613816288 0.0006403953404404278 0.02461729439488529" rpy="0 0 0"/>
+    <mass value="0.024732672038933038"/>
+    <inertia ixx="9e-06" iyy="1.3e-05" izz="1.8e-05" ixy="4e-06" iyz="2e-06" ixz="-3e-06"/>
   </inertial>
   <visual>
     <origin xyz="-0.292144 0.096267 -0.108" rpy="0 0 0"/>
     <geometry>
-      <mesh filename="package://assembly_main_description/meshes/hand_finger_v2_1.stl" scale="0.001 0.001 0.001"/>
-    </geometry>
-    <material name="steel_satin"/>
+      <mesh filename="package://assembly_main_description/meshes/hand_finger_v6_1.stl" scale="0.001 0.001 0.001"/>
+    </geometry>
+    <material name="abs_white"/>
   </visual>
   <collision>
     <origin xyz="-0.292144 0.096267 -0.108" rpy="0 0 0"/>
     <geometry>
-      <mesh filename="package://assembly_main_description/meshes/hand_finger_v2_1.stl" scale="0.001 0.001 0.001"/>
+      <mesh filename="package://assembly_main_description/meshes/hand_finger_v6_1.stl" scale="0.001 0.001 0.001"/>
     </geometry>
   </collision>
@@ -291,10 +291,10 @@
   <origin xyz="0.017558 0.001411 0.04" rpy="0 0 0"/>
   <parent link="arm_bracket_temp_v12_1"/>
-  <child link="arm_root_v1_1"/>
+  <child link="arm_root_v4_1"/>
 </joint>
 <joint name="Revolute 1" type="revolute">
   <origin xyz="0.03568 -0.0206 0.01305" rpy="0 0 0"/>
-  <parent link="arm_root_v1_1"/>
-  <child link="pitch_1_test_v1_1"/>
+  <parent link="arm_root_v4_1"/>
+  <child link="pitch_1_test_v3_1"/>
   <axis xyz="-0.0 0.0 -1.0"/>
   <limit upper="1.570796" lower="-1.570796" effort="100" velocity="100"/>
@@ -302,6 +302,6 @@
 <joint name="Revolute_2" type="revolute">
   <origin xyz="0.043692 -0.048724 0.00545" rpy="0 0 0"/>
-  <parent link="pitch_1_test_v1_1"/>
-  <child link="roll_1_test_v1_1"/>
+  <parent link="pitch_1_test_v3_1"/>
+  <child link="roll_1_test_v3_1"/>
   <axis xyz="0.5 0.866025 -0.0"/>
   <limit upper="1.919862" lower="-1.396263" effort="100" velocity="100"/>
@@ -309,12 +309,12 @@
 <joint name="Revolute_3" type="continuous">
   <origin xyz="0.059443 -0.00984 0.0" rpy="0 0 0"/>
-  <parent link="roll_1_test_v1_1"/>
-  <child link="pitch_2_test_v1_1"/>
+  <parent link="roll_1_test_v3_1"/>
+  <child link="pitch_2_test_v3_1"/>
   <axis xyz="0.866025 -0.5 0.0"/>
 </joint>
 <joint name="Revolute_4" type="revolute">
   <origin xyz="0.029511 -0.041287 0.0" rpy="0 0 0"/>
-  <parent link="pitch_2_test_v1_1"/>
-  <child link="roll_2_test_v1_1"/>
+  <parent link="pitch_2_test_v3_1"/>
+  <child link="roll_2_test_v3_1"/>
   <axis xyz="0.5 0.866025 0.0"/>
   <limit upper="1.919862" lower="-1.48353" effort="100" velocity="100"/>
@@ -322,12 +322,12 @@
 <joint name="Revolute_5" type="continuous">
   <origin xyz="0.059444 -0.00984 0.0" rpy="0 0 0"/>
-  <parent link="roll_2_test_v1_1"/>
-  <child link="hand_unit_v1_1"/>
+  <parent link="roll_2_test_v3_1"/>
+  <child link="hand_unit_v3_1"/>
   <axis xyz="-0.866025 0.5 -0.0"/>
 </joint>
 <joint name="Revolute_6" type="revolute">
   <origin xyz="0.011113 -0.032051 0.013" rpy="0 0 0"/>
-  <parent link="hand_unit_v1_1"/>
-  <child link="hand_finger_v2_1"/>
+  <parent link="hand_unit_v3_1"/>
+  <child link="hand_finger_v6_1"/>
   <axis xyz="0.5 0.866025 0.0"/>
   <limit upper="0.872665" lower="-1.047198" effort="100" velocity="100"/>

File: urdf/komarm.urdf (robot description, URDF)
Before this commit: robot assembly_main, 13 links, 12 joints
Links:
- removed link arm_root_v1_1
- removed link hand_finger_v2_1
- removed link hand_unit_v1_1
- removed link pitch_1_test_v1_1
- removed link pitch_2_test_v1_1
- removed link roll_1_test_v1_1
- removed link roll_2_test_v1_1
- added link arm_root_v4_1, mass 0.06457976620923557; collision mesh filename=../meshes/arm_root_v4_1.stl scale=0.001 0.001 0.001; visual mesh filename=../meshes/arm_root_v4_1.stl scale=0.001 0.001 0.001
- added link hand_finger_v6_1, mass 0.024732672038933038; collision mesh filename=../meshes/hand_finger_v6_1.stl scale=0.001 0.001 0.001; visual mesh filename=../meshes/hand_finger_v6_1.stl scale=0.001 0.001 0.001
- added link hand_unit_v3_1, mass 0.0952280970557457; collision mesh filename=../meshes/hand_unit_v3_1.stl scale=0.001 0.001 0.001; visual mesh filename=../meshes/hand_unit_v3_1.stl scale=0.001 0.001 0.001
- added link pitch_1_test_v3_1, mass 0.08186133563123103; collision mesh filename=../meshes/pitch_1_test_v3_1.stl scale=0.001 0.001 0.001; visual mesh filename=../meshes/pitch_1_test_v3_1.stl scale=0.001 0.001 0.001
- added link pitch_2_test_v3_1, mass 0.06668343069893205; collision mesh filename=../meshes/pitch_2_test_v3_1.stl scale=0.001 0.001 0.001; visual mesh filename=../meshes/pitch_2_test_v3_1.stl scale=0.001 0.001 0.001
- added link roll_1_test_v3_1, mass 0.07353297901744495; collision mesh filename=../meshes/roll_1_test_v3_1.stl scale=0.001 0.001 0.001; visual mesh filename=../meshes/roll_1_test_v3_1.stl scale=0.001 0.001 0.001
- added link roll_2_test_v3_1, mass 0.07365581710871624; collision mesh filename=../meshes/roll_2_test_v3_1.stl scale=0.001 0.001 0.001; visual mesh filename=../meshes/roll_2_test_v3_1.stl scale=0.001 0.001 0.001
- link base_link: mass 20.0 -> 10.0
Joints:
- removed joint Revolute_1
- added joint Revolute 1: type revolute, parent arm_root_v4_1, child pitch_1_test_v3_1, origin xyz=0.03568 -0.0206 0.01305 rpy=0 0 0, axis -0.0 0.0 -1.0, limit lower=-1.570796 upper=1.570796 effort=100 velocity=100
- joint Revolute_2: child roll_1_test_v1_1 -> roll_1_test_v3_1; parent pitch_1_test_v1_1 -> pitch_1_test_v3_1
- joint Revolute_3: child pitch_2_test_v1_1 -> pitch_2_test_v3_1; parent roll_1_test_v1_1 -> roll_1_test_v3_1
- joint Revolute_4: child roll_2_test_v1_1 -> roll_2_test_v3_1; parent pitch_2_test_v1_1 -> pitch_2_test_v3_1
- joint Revolute_5: child hand_unit_v1_1 -> hand_unit_v3_1; parent roll_2_test_v1_1 -> roll_2_test_v3_1
- joint Revolute_6: child hand_finger_v2_1 -> hand_finger_v6_1; parent hand_unit_v1_1 -> hand_unit_v3_1
- joint Rigid 26: child arm_root_v1_1 -> arm_root_v4_1

File: urdf/materials.xacro (robot description, xacro)
@@ -10,3 +10,6 @@
   <color rgba="0.9607843137254902 0.9607843137254902 0.9647058823529412 1.0"/>
 </material>
+<material name="abs_white">
+  <color rgba="0.9647058823529412 0.9647058823529412 0.9529411764705882 1.0"/>
+</material>
 </robot>
