Commit message: fix(urdf): home position and orientation

File: urdf/assembly_main.xacro (robot description, xacro)
@@ -5,7 +5,7 @@
 <link name="base_link">
   <inertial>
-    <origin xyz="0.0016685480823734394 0.09587231603609693 0.01410222124869956" rpy="0 0 0"/>
-    <mass value="4.116732793254999"/>
-    <inertia ixx="0.013163" iyy="0.013452" izz="0.024089" ixy="0.000254" iyz="2.5e-05" ixz="-4.4e-05"/>
+    <origin xyz="0.001924209931808292 9.588003529118677e-06 -0.017397201457223316" rpy="0 0 0"/>
+    <mass value="10.00"/>
+    <inertia ixx="0.013016" iyy="0.013601" izz="0.02409" ixy="2e-06" iyz="-1e-06" ixz="-5.1e-05"/>
   </inertial>
   <visual>
@@ -25,10 +25,10 @@
 <link name="arm_bracket_temp_v12_1">
   <inertial>
-    <origin xyz="0.011893307409353286 0.004680842759964748 0.022739357849046002" rpy="0 0 0"/>
+    <origin xyz="0.007959481790445908 0.009999999999998583 0.02273935784904592" rpy="0 0 0"/>
     <mass value="0.16496925038992882"/>
-    <inertia ixx="9e-05" iyy="7e-05" izz="5.2e-05" ixy="-1.7e-05" iyz="5e-06" ixz="-8e-06"/>
-  </inertial>
-  <visual>
-    <origin xyz="-0.035703 -0.064664 -0.0365" rpy="0 0 0"/>
+    <inertia ixx="9.9e-05" iyy="6.1e-05" izz="5.2e-05" ixy="-0.0" iyz="-0.0" ixz="-1e-05"/>
+  </inertial>
+  <visual>
+    <origin xyz="-0.047 0.01 -0.005" rpy="0 0 0"/>
     <geometry>
       <mesh filename="package://assembly_main_description/meshes/arm_bracket_temp_v12_1.stl" scale="0.001 0.001 0.001"/>
@@ -37,5 +37,5 @@
   </visual>
   <collision>
-    <origin xyz="-0.035703 -0.064664 -0.0365" rpy="0 0 0"/>
+    <origin xyz="-0.047 0.01 -0.005" rpy="0 0 0"/>
     <geometry>
       <mesh filename="package://assembly_main_description/meshes/arm_bracket_temp_v12_1.stl" scale="0.001 0.001 0.001"/>
@@ -45,10 +45,10 @@
 <link name="raspi4_bracket_v1_1">
   <inertial>
-    <origin xyz="1.0358811586286266e-11 -0.004190801342254108 0.011212626337856427" rpy="0 0 0"/>
+    <origin xyz="0.0020951925076898026 -0.0036289475514907216 0.011212626337856312" rpy="0 0 0"/>
     <mass value="0.10292684148685698"/>
-    <inertia ixx="2e-05" iyy="4.1e-05" izz="4.4e-05" ixy="0.0" iyz="4e-06" ixz="-0.0"/>
-  </inertial>
-  <visual>
-    <origin xyz="-0.0 -0.176825 -0.0365" rpy="0 0 0"/>
+    <inertia ixx="2.6e-05" iyy="3.6e-05" izz="4.4e-05" ixy="-9e-06" iyz="4e-06" ixz="-2e-06"/>
+  </inertial>
+  <visual>
+    <origin xyz="0.04 -0.069282 -0.005" rpy="0 0 0"/>
     <geometry>
       <mesh filename="package://assembly_main_description/meshes/raspi4_bracket_v1_1.stl" scale="0.001 0.001 0.001"/>
@@ -57,5 +57,5 @@
   </visual>
   <collision>
-    <origin xyz="-0.0 -0.176825 -0.0365" rpy="0 0 0"/>
+    <origin xyz="0.04 -0.069282 -0.005" rpy="0 0 0"/>
     <geometry>
       <mesh filename="package://assembly_main_description/meshes/raspi4_bracket_v1_1.stl" scale="0.001 0.001 0.001"/>
@@ -65,10 +65,10 @@
 <link name="raspi4_v2_1">
   <inertial>
-    <origin xyz="3.881339694089547e-15 0.014999583655189608 0.03859010164223097" rpy="0 0 0"/>
+    <origin xyz="-0.00749999999999993 0.01299008311032395 0.038590101642230826" rpy="0 0 0"/>
     <mass value="0.7390104624417327"/>
-    <inertia ixx="0.000465" iyy="0.000631" izz="0.000215" ixy="0.0" iyz="0.0" ixz="1e-06"/>
-  </inertial>
-  <visual>
-    <origin xyz="-0.0 -0.163825 -0.0575" rpy="0 0 0"/>
+    <inertia ixx="0.000507" iyy="0.00059" izz="0.000215" ixy="-7.2e-05" iyz="1e-06" ixz="1e-06"/>
+  </inertial>
+  <visual>
+    <origin xyz="0.0335 -0.058024 -0.026" rpy="0 0 0"/>
     <geometry>
       <mesh filename="package://assembly_main_description/meshes/raspi4_v2_1.stl" scale="0.001 0.001 0.001"/>
@@ -77,5 +77,5 @@
   </visual>
   <collision>
-    <origin xyz="-0.0 -0.163825 -0.0575" rpy="0 0 0"/>
+    <origin xyz="0.0335 -0.058024 -0.026" rpy="0 0 0"/>
     <geometry>
       <mesh filename="package://assembly_main_description/meshes/raspi4_v2_1.stl" scale="0.001 0.001 0.001"/>
@@ -85,10 +85,10 @@
 <link name="lipo_bracket_v5_1">
   <inertial>
-    <origin xyz="-0.02145046736939967 -0.02300777254127473 0.025572386759107592" rpy="0 0 0"/>
+    <origin xyz="-0.007072287607066324 -0.03064999999999981 0.02557238675910756" rpy="0 0 0"/>
     <mass value="0.15095338739595293"/>
-    <inertia ixx="0.000129" iyy="0.000116" izz="9.8e-05" ixy="-1.2e-05" iyz="-0.0" ixz="1e-06"/>
-  </inertial>
-  <visual>
-    <origin xyz="0.040468 -0.155581 -0.0365" rpy="0 0 0"/>
+    <inertia ixx="0.000136" iyy="0.000109" izz="9.8e-05" ixy="-0.0" iyz="0.0" ixz="1e-06"/>
+  </inertial>
+  <visual>
+    <origin xyz="0.064425 -0.03065 -0.005" rpy="0 0 0"/>
     <geometry>
       <mesh filename="package://assembly_main_description/meshes/lipo_bracket_v5_1.stl" scale="0.001 0.001 0.001"/>
@@ -97,5 +97,5 @@
   </visual>
   <collision>
-    <origin xyz="0.040468 -0.155581 -0.0365" rpy="0 0 0"/>
+    <origin xyz="0.064425 -0.03065 -0.005" rpy="0 0 0"/>
     <geometry>
       <mesh filename="package://assembly_main_description/meshes/lipo_bracket_v5_1.stl" scale="0.001 0.001 0.001"/>
@@ -105,10 +105,10 @@
 <link name="DZ47B_63_circuit_breaker_holder_v3_1">
   <inertial>
-    <origin xyz="0.02229875370121319 -0.03862280991922731 0.002938007686629586" rpy="0 0 0"/>
+    <origin xyz="0.03862239340692045 -0.022298666174134715 0.0029380076866297187" rpy="0 0 0"/>
     <mass value="0.012274791356152887"/>
-    <inertia ixx="1.5e-05" iyy="5e-06" izz="2e-05" ixy="8e-06" iyz="0.0" ixz="-0.0"/>
-  </inertial>
-  <visual>
-    <origin xyz="0.088434 -0.095997 -0.0365" rpy="0 0 0"/>
+    <inertia ixx="5e-06" iyy="1.5e-05" izz="2e-05" ixy="8e-06" iyz="0.0" ixz="-0.0"/>
+  </inertial>
+  <visual>
+    <origin xyz="0.076172 0.044934 -0.005" rpy="0 0 0"/>
     <geometry>
       <mesh filename="package://assembly_main_description/meshes/DZ47B_63_circuit_breaker_holder_v3_1.stl" scale="0.001 0.001 0.001"/>
@@ -117,5 +117,5 @@
   </visual>
   <collision>
-    <origin xyz="0.088434 -0.095997 -0.0365" rpy="0 0 0"/>
+    <origin xyz="0.076172 0.044934 -0.005" rpy="0 0 0"/>
     <geometry>
       <mesh filename="package://assembly_main_description/meshes/DZ47B_63_circuit_breaker_holder_v3_1.stl" scale="0.001 0.001 0.001"/>
@@ -125,10 +125,10 @@
 <link name="arm_root_v4_1">
   <inertial>
-    <origin xyz="0.022163724443126365 -0.012796901291084212 -0.009138901606431687" rpy="0 0 0"/>
+    <origin xyz="0.02559296991432554 1.2574053551176077e-11 -0.009138901606431792" rpy="0 0 0"/>
     <mass value="0.06457976620923557"/>
-    <inertia ixx="1.6e-05" iyy="2.1e-05" izz="1.9e-05" ixy="5e-06" iyz="0.0" ixz="-1e-06"/>
-  </inertial>
-  <visual>
-    <origin xyz="-0.053261 -0.066075 -0.0765" rpy="0 0 0"/>
+    <inertia ixx="1.3e-05" iyy="2.4e-05" izz="1.9e-05" ixy="0.0" iyz="0.0" ixz="-1e-06"/>
+  </inertial>
+  <visual>
+    <origin xyz="-0.0615 -0.0 -0.045" rpy="0 0 0"/>
     <geometry>
       <mesh filename="package://assembly_main_description/meshes/arm_root_v4_1.stl" scale="0.001 0.001 0.001"/>
@@ -137,5 +137,5 @@
   </visual>
   <collision>
-    <origin xyz="-0.053261 -0.066075 -0.0765" rpy="0 0 0"/>
+    <origin xyz="-0.0615 -0.0 -0.045" rpy="0 0 0"/>
     <geometry>
       <mesh filename="package://assembly_main_description/meshes/arm_root_v4_1.stl" scale="0.001 0.001 0.001"/>
@@ -145,10 +145,10 @@
 <link name="pitch_1_test_v3_1">
   <inertial>
-    <origin xyz="0.0358303038564968 -0.019899545668259706 -0.00013072073296151177" rpy="0 0 0"/>
+    <origin xyz="0.04097968346475826 0.0006820959366182021 -0.0001307207329616436" rpy="0 0 0"/>
     <mass value="0.08186133563123103"/>
-    <inertia ixx="3e-05" iyy="4e-05" izz="3.7e-05" ixy="6e-06" iyz="5e-06" ixz="-9e-06"/>
-  </inertial>
-  <visual>
-    <origin xyz="-0.088941 -0.045475 -0.08955" rpy="0 0 0"/>
+    <inertia ixx="2.7e-05" iyy="4.3e-05" izz="3.7e-05" ixy="-1e-06" iyz="-0.0" ixz="-1e-05"/>
+  </inertial>
+  <visual>
+    <origin xyz="-0.1027 0.0 -0.05805" rpy="0 0 0"/>
     <geometry>
       <mesh filename="package://assembly_main_description/meshes/pitch_1_test_v3_1.stl" scale="0.001 0.001 0.001"/>
@@ -157,5 +157,5 @@
   </visual>
   <collision>
-    <origin xyz="-0.088941 -0.045475 -0.08955" rpy="0 0 0"/>
+    <origin xyz="-0.1027 0.0 -0.05805" rpy="0 0 0"/>
     <geometry>
       <mesh filename="package://assembly_main_description/meshes/pitch_1_test_v3_1.stl" scale="0.001 0.001 0.001"/>
@@ -165,10 +165,10 @@
 <link name="roll_1_test_v3_1">
   <inertial>
-    <origin xyz="0.042100640863960814 0.00017256453450652937 0.015160914691842262" rpy="0 0 0"/>
+    <origin xyz="0.0363742814442784 0.0212000000095127 0.015160914691842164" rpy="0 0 0"/>
     <mass value="0.07353297901744495"/>
-    <inertia ixx="2.5e-05" iyy="2.7e-05" izz="2.1e-05" ixy="2e-06" iyz="0.0" ixz="-0.0"/>
-  </inertial>
-  <visual>
-    <origin xyz="-0.132633 0.003249 -0.095" rpy="0 0 0"/>
+    <inertia ixx="2.4e-05" iyy="2.9e-05" izz="2.1e-05" ixy="0.0" iyz="-0.0" ixz="-1e-06"/>
+  </inertial>
+  <visual>
+    <origin xyz="-0.1649 0.02035 -0.0635" rpy="0 0 0"/>
     <geometry>
       <mesh filename="package://assembly_main_description/meshes/roll_1_test_v3_1.stl" scale="0.001 0.001 0.001"/>
@@ -177,5 +177,5 @@
   </visual>
   <collision>
-    <origin xyz="-0.132633 0.003249 -0.095" rpy="0 0 0"/>
+    <origin xyz="-0.1649 0.02035 -0.0635" rpy="0 0 0"/>
     <geometry>
       <mesh filename="package://assembly_main_description/meshes/roll_1_test_v3_1.stl" scale="0.001 0.001 0.001"/>
@@ -185,10 +185,10 @@
 <link name="pitch_2_test_v3_1">
   <inertial>
-    <origin xyz="0.025973068908376362 -0.014769408547619371 -2.946918264967735e-10" rpy="0 0 0"/>
+    <origin xyz="0.029877529047602214 0.0001958957866964999 -2.9469195139686377e-10" rpy="0 0 0"/>
     <mass value="0.06668343069893205"/>
-    <inertia ixx="1.5e-05" iyy="1.9e-05" izz="2.6e-05" ixy="2e-06" iyz="0.0" ixz="-0.0"/>
-  </inertial>
-  <visual>
-    <origin xyz="-0.192076 0.013089 -0.095" rpy="0 0 0"/>
+    <inertia ixx="1.4e-05" iyy="2e-05" izz="2.6e-05" ixy="-1e-06" iyz="-0.0" ixz="-0.0"/>
+  </inertial>
+  <visual>
+    <origin xyz="-0.2213 -0.00085 -0.0635" rpy="0 0 0"/>
     <geometry>
       <mesh filename="package://assembly_main_description/meshes/pitch_2_test_v3_1.stl" scale="0.001 0.001 0.001"/>
@@ -197,5 +197,5 @@
   </visual>
   <collision>
-    <origin xyz="-0.192076 0.013089 -0.095" rpy="0 0 0"/>
+    <origin xyz="-0.2213 -0.00085 -0.0635" rpy="0 0 0"/>
     <geometry>
       <mesh filename="package://assembly_main_description/meshes/pitch_2_test_v3_1.stl" scale="0.001 0.001 0.001"/>
@@ -205,10 +205,10 @@
 <link name="roll_2_test_v3_1">
   <inertial>
-    <origin xyz="0.04210189544568463 0.000172164463575597 0.015187663571532464" rpy="0 0 0"/>
+    <origin xyz="0.036375491747628774 0.021200000009496393 0.015187663571532395" rpy="0 0 0"/>
     <mass value="0.07365581710871624"/>
-    <inertia ixx="2.5e-05" iyy="2.7e-05" izz="2.1e-05" ixy="2e-06" iyz="0.0" ixz="-0.0"/>
-  </inertial>
-  <visual>
-    <origin xyz="-0.221587 0.054376 -0.095" rpy="0 0 0"/>
+    <inertia ixx="2.4e-05" iyy="2.9e-05" izz="2.1e-05" ixy="0.0" iyz="-0.0" ixz="-1e-06"/>
+  </inertial>
+  <visual>
+    <origin xyz="-0.2675 0.02015 -0.0635" rpy="0 0 0"/>
     <geometry>
       <mesh filename="package://assembly_main_description/meshes/roll_2_test_v3_1.stl" scale="0.001 0.001 0.001"/>
@@ -217,5 +217,5 @@
   </visual>
   <collision>
-    <origin xyz="-0.221587 0.054376 -0.095" rpy="0 0 0"/>
+    <origin xyz="-0.2675 0.02015 -0.0635" rpy="0 0 0"/>
     <geometry>
       <mesh filename="package://assembly_main_description/meshes/roll_2_test_v3_1.stl" scale="0.001 0.001 0.001"/>
@@ -225,10 +225,10 @@
 <link name="hand_unit_v3_1">
   <inertial>
-    <origin xyz="0.027318565725242272 -0.01604965279786605 -0.011102966860764008" rpy="0 0 0"/>
+    <origin xyz="0.031683675390487276 -0.00023986066792197516 -0.011102966860764112" rpy="0 0 0"/>
     <mass value="0.0952280970557457"/>
-    <inertia ixx="5.4e-05" iyy="6.8e-05" izz="5.4e-05" ixy="1.1e-05" iyz="-8e-06" ixz="1.7e-05"/>
-  </inertial>
-  <visual>
-    <origin xyz="-0.281031 0.064216 -0.095" rpy="0 0 0"/>
+    <inertia ixx="4.8e-05" iyy="7.4e-05" izz="5.4e-05" ixy="-0.0" iyz="1e-06" ixz="1.9e-05"/>
+  </inertial>
+  <visual>
+    <origin xyz="-0.3239 -0.00105 -0.0635" rpy="0 0 0"/>
     <geometry>
       <mesh filename="package://assembly_main_description/meshes/hand_unit_v3_1.stl" scale="0.001 0.001 0.001"/>
@@ -237,5 +237,5 @@
   </visual>
   <collision>
-    <origin xyz="-0.281031 0.064216 -0.095" rpy="0 0 0"/>
+    <origin xyz="-0.3239 -0.00105 -0.0635" rpy="0 0 0"/>
     <geometry>
       <mesh filename="package://assembly_main_description/meshes/hand_unit_v3_1.stl" scale="0.001 0.001 0.001"/>
@@ -243,92 +243,92 @@
   </collision>
 </link>
-<link name="hand_finger_v6_1">
-  <inertial>
-    <origin xyz="0.04229123613816288 0.0006403953404404278 0.02461729439488529" rpy="0 0 0"/>
+<link name="hand_finger_v7_1">
+  <inertial>
+    <origin xyz="0.03630500457367125 0.02170000000000132 0.024617294394885247" rpy="0 0 0"/>
     <mass value="0.024732672038933038"/>
-    <inertia ixx="9e-06" iyy="1.3e-05" izz="1.8e-05" ixy="4e-06" iyz="2e-06" ixz="-3e-06"/>
-  </inertial>
-  <visual>
-    <origin xyz="-0.292144 0.096267 -0.108" rpy="0 0 0"/>
-    <geometry>
-      <mesh filename="package://assembly_main_description/meshes/hand_finger_v6_1.stl" scale="0.001 0.001 0.001"/>
-    </geometry>
-    <material name="abs_white"/>
-  </visual>
-  <collision>
-    <origin xyz="-0.292144 0.096267 -0.108" rpy="0 0 0"/>
-    <geometry>
-      <mesh filename="package://assembly_main_description/meshes/hand_finger_v6_1.stl" scale="0.001 0.001 0.001"/>
+    <inertia ixx="7e-06" iyy="1.5e-05" izz="1.8e-05" ixy="-0.0" iyz="0.0" ixz="-4e-06"/>
+  </inertial>
+  <visual>
+    <origin xyz="-0.34955 0.02115 -0.0765" rpy="0 0 0"/>
+    <geometry>
+      <mesh filename="package://assembly_main_description/meshes/hand_finger_v7_1.stl" scale="0.001 0.001 0.001"/>
+    </geometry>
+    <material name="abs_white"/>
+  </visual>
+  <collision>
+    <origin xyz="-0.34955 0.02115 -0.0765" rpy="0 0 0"/>
+    <geometry>
+      <mesh filename="package://assembly_main_description/meshes/hand_finger_v7_1.stl" scale="0.001 0.001 0.001"/>
     </geometry>
   </collision>
 </link>
 <joint name="Rigid 4" type="fixed">
-  <origin xyz="0.035703 0.064664 0.0365" rpy="0 0 0"/>
+  <origin xyz="0.047 -0.01 0.005" rpy="0 0 0"/>
   <parent link="base_link"/>
   <child link="arm_bracket_temp_v12_1"/>
 </joint>
 <joint name="Rigid 7" type="fixed">
-  <origin xyz="0.0 0.176825 0.0365" rpy="0 0 0"/>
+  <origin xyz="-0.04 0.069282 0.005" rpy="0 0 0"/>
   <parent link="base_link"/>
   <child link="raspi4_bracket_v1_1"/>
 </joint>
 <joint name="Rigid 8" type="fixed">
-  <origin xyz="0.0 -0.013 0.021" rpy="0 0 0"/>
+  <origin xyz="0.0065 -0.011258 0.021" rpy="0 0 0"/>
   <parent link="raspi4_bracket_v1_1"/>
   <child link="raspi4_v2_1"/>
 </joint>
 <joint name="Rigid 16" type="fixed">
-  <origin xyz="-0.040468 0.155581 0.0365" rpy="0 0 0"/>
+  <origin xyz="-0.064425 0.03065 0.005" rpy="0 0 0"/>
   <parent link="base_link"/>
   <child link="lipo_bracket_v5_1"/>
 </joint>
 <joint name="Rigid 17" type="fixed">
-  <origin xyz="-0.088434 0.095997 0.0365" rpy="0 0 0"/>
+  <origin xyz="-0.076172 -0.044934 0.005" rpy="0 0 0"/>
   <parent link="base_link"/>
   <child link="DZ47B_63_circuit_breaker_holder_v3_1"/>
 </joint>
 <joint name="Rigid 26" type="fixed">
-  <origin xyz="0.017558 0.001411 0.04" rpy="0 0 0"/>
+  <origin xyz="0.0145 0.01 0.04" rpy="0 0 0"/>
   <parent link="arm_bracket_temp_v12_1"/>
   <child link="arm_root_v4_1"/>
 </joint>
-<joint name="Revolute 1" type="revolute">
-  <origin xyz="0.03568 -0.0206 0.01305" rpy="0 0 0"/>
+<joint name="Revolute_1" type="revolute">
+  <origin xyz="0.0412 -0.0 0.01305" rpy="0 0 0"/>
   <parent link="arm_root_v4_1"/>
   <child link="pitch_1_test_v3_1"/>
-  <axis xyz="-0.0 0.0 -1.0"/>
+  <axis xyz="0.0 -0.0 -1.0"/>
   <limit upper="1.570796" lower="-1.570796" effort="100" velocity="100"/>
 </joint>
 <joint name="Revolute_2" type="revolute">
-  <origin xyz="0.043692 -0.048724 0.00545" rpy="0 0 0"/>
+  <origin xyz="0.0622 -0.02035 0.00545" rpy="0 0 0"/>
   <parent link="pitch_1_test_v3_1"/>
   <child link="roll_1_test_v3_1"/>
-  <axis xyz="0.5 0.866025 -0.0"/>
+  <axis xyz="-0.0 1.0 -0.0"/>
   <limit upper="1.919862" lower="-1.396263" effort="100" velocity="100"/>
 </joint>
 <joint name="Revolute_3" type="continuous">
-  <origin xyz="0.059443 -0.00984 0.0" rpy="0 0 0"/>
+  <origin xyz="0.0564 0.0212 0.0" rpy="0 0 0"/>
   <parent link="roll_1_test_v3_1"/>
   <child link="pitch_2_test_v3_1"/>
-  <axis xyz="0.866025 -0.5 0.0"/>
+  <axis xyz="1.0 0.0 0.0"/>
 </joint>
 <joint name="Revolute_4" type="revolute">
-  <origin xyz="0.029511 -0.041287 0.0" rpy="0 0 0"/>
+  <origin xyz="0.0462 -0.021 0.0" rpy="0 0 0"/>
   <parent link="pitch_2_test_v3_1"/>
   <child link="roll_2_test_v3_1"/>
-  <axis xyz="0.5 0.866025 0.0"/>
+  <axis xyz="-0.0 1.0 0.0"/>
   <limit upper="1.919862" lower="-1.48353" effort="100" velocity="100"/>
 </joint>
 <joint name="Revolute_5" type="continuous">
-  <origin xyz="0.059444 -0.00984 0.0" rpy="0 0 0"/>
+  <origin xyz="0.0564 0.0212 0.0" rpy="0 0 0"/>
   <parent link="roll_2_test_v3_1"/>
   <child link="hand_unit_v3_1"/>
-  <axis xyz="-0.866025 0.5 -0.0"/>
+  <axis xyz="-1.0 0.0 -0.0"/>
 </joint>
 <joint name="Revolute_6" type="revolute">
-  <origin xyz="0.011113 -0.032051 0.013" rpy="0 0 0"/>
+  <origin xyz="0.02565 -0.0222 0.013" rpy="0 0 0"/>
   <parent link="hand_unit_v3_1"/>
-  <child link="hand_finger_v6_1"/>
-  <axis xyz="0.5 0.866025 0.0"/>
+  <child link="hand_finger_v7_1"/>
+  <axis xyz="0.0 1.0 -0.0"/>
   <limit upper="0.872665" lower="-1.047198" effort="100" velocity="100"/>
 </joint>

File: urdf/komarm.urdf (robot description, URDF)
Before this commit: robot assembly_main, 13 links, 12 joints
Links:
- removed link hand_finger_v6_1
- added link hand_finger_v7_1, mass 0.024732672038933038; collision mesh filename=../meshes/hand_finger_v7_1.stl scale=0.001 0.001 0.001; visual mesh filename=../meshes/hand_finger_v7_1.stl scale=0.001 0.001 0.001
- link base_link: mass 10.0 -> 10.00
Joints:
- joint Revolute_1: axis -0.0 0.0 -1.0 -> 0.0 -0.0 -1.0; origin xyz=0.03568 -0.0206 0.01305 rpy=0 0 0 -> xyz=0.0412 -0.0 0.01305 rpy=0 0 0
- joint Revolute_2: axis 0.5 0.866025 -0.0 -> -0.0 1.0 -0.0; origin xyz=0.043692 -0.048724 0.00545 rpy=0 0 0 -> xyz=0.0622 -0.02035 0.00545 rpy=0 0 0
- joint Revolute_3: axis 0.866025 -0.5 0.0 -> 1.0 0.0 0.0; origin xyz=0.059443 -0.00984 0.0 rpy=0 0 0 -> xyz=0.0564 0.0212 0.0 rpy=0 0 0
- joint Revolute_4: axis 0.5 0.866025 0.0 -> -0.0 1.0 0.0; origin xyz=0.029511 -0.041287 0.0 rpy=0 0 0 -> xyz=0.0462 -0.021 0.0 rpy=0 0 0
- joint Revolute_5: axis -0.866025 0.5 -0.0 -> -1.0 0.0 -0.0; origin xyz=0.059444 -0.00984 0.0 rpy=0 0 0 -> xyz=0.0564 0.0212 0.0 rpy=0 0 0
- joint Revolute_6: axis 0.5 0.866025 0.0 -> 0.0 1.0 -0.0; child hand_finger_v6_1 -> hand_finger_v7_1; origin xyz=0.011113 -0.032051 0.013 rpy=0 0 0 -> xyz=0.02565 -0.0222 0.013 rpy=0 0 0
- joint Rigid 16: origin xyz=-0.040468 0.155581 0.0365 rpy=0 0 0 -> xyz=-0.064425 0.03065 0.005 rpy=0 0 0
- joint Rigid 17: origin xyz=-0.088434 0.095997 0.0365 rpy=0 0 0 -> xyz=-0.076172 -0.044934 0.005 rpy=0 0 0
- joint Rigid 26: origin xyz=0.017558 0.001411 0.04 rpy=0 0 0 -> xyz=0.0145 0.01 0.04 rpy=0 0 0
- joint Rigid 4: origin xyz=0.035703 0.064664 0.0365 rpy=0 0 0 -> xyz=0.047 -0.01 0.005 rpy=0 0 0
- joint Rigid 7: origin xyz=0.0 0.176825 0.0365 rpy=0 0 0 -> xyz=-0.04 0.069282 0.005 rpy=0 0 0
- joint Rigid 8: origin xyz=0.0 -0.013 0.021 rpy=0 0 0 -> xyz=0.0065 -0.011258 0.021 rpy=0 0 0
