Commit message: feat(urdf): update

File: urdf/assembly_main.xacro (robot description, xacro)
@@ -5,7 +5,7 @@
 <link name="base_link">
   <inertial>
-    <origin xyz="0.001924209931808292 9.588003529118677e-06 -0.017397201457223316" rpy="0 0 0"/>
-    <mass value="10.00"/>
-    <inertia ixx="0.013016" iyy="0.013601" izz="0.02409" ixy="2e-06" iyz="-1e-06" ixz="-5.1e-05"/>
+    <origin xyz="0.005188065648430864 -0.00026933142160205393 -0.01663287964245459" rpy="0 0 0"/>
+    <mass value="4.27590428722208"/>
+    <inertia ixx="0.013169" iyy="0.014957" izz="0.025457" ixy="0.000108" iyz="2.4e-05" ixz="-0.000335"/>
   </inertial>
   <visual>
@@ -14,5 +14,5 @@
       <mesh filename="package://assembly_main_description/meshes/base_link.stl" scale="0.001 0.001 0.001"/>
     </geometry>
-    <material name="aluminum_satin"/>
+    <material name="opaque141141141"/>
   </visual>
   <collision>
@@ -23,34 +23,34 @@
   </collision>
 </link>
-<link name="arm_bracket_temp_v12_1">
-  <inertial>
-    <origin xyz="0.007959481790445908 0.009999999999998583 0.02273935784904592" rpy="0 0 0"/>
-    <mass value="0.16496925038992882"/>
-    <inertia ixx="9.9e-05" iyy="6.1e-05" izz="5.2e-05" ixy="-0.0" iyz="-0.0" ixz="-1e-05"/>
-  </inertial>
-  <visual>
-    <origin xyz="-0.047 0.01 -0.005" rpy="0 0 0"/>
-    <geometry>
-      <mesh filename="package://assembly_main_description/meshes/arm_bracket_temp_v12_1.stl" scale="0.001 0.001 0.001"/>
-    </geometry>
-    <material name="steel_satin"/>
-  </visual>
-  <collision>
-    <origin xyz="-0.047 0.01 -0.005" rpy="0 0 0"/>
-    <geometry>
-      <mesh filename="package://assembly_main_description/meshes/arm_bracket_temp_v12_1.stl" scale="0.001 0.001 0.001"/>
-    </geometry>
-  </collision>
-</link>
-<link name="raspi4_bracket_v1_1">
-  <inertial>
-    <origin xyz="0.0020951925076898026 -0.0036289475514907216 0.011212626337856312" rpy="0 0 0"/>
-    <mass value="0.10292684148685698"/>
-    <inertia ixx="2.6e-05" iyy="3.6e-05" izz="4.4e-05" ixy="-9e-06" iyz="4e-06" ixz="-2e-06"/>
+<link name="wheel_control_board_v7_2">
+  <inertial>
+    <origin xyz="0.021526332400288135 -0.034185196183547054 0.10000262508964397" rpy="0 0 0"/>
+    <mass value="0.05597515361092653"/>
+    <inertia ixx="3.1e-05" iyy="1e-05" izz="4e-05" ixy="1e-06" iyz="-0.0" ixz="-0.0"/>
+  </inertial>
+  <visual>
+    <origin xyz="0.025 -0.0292 -0.0116" rpy="0 0 0"/>
+    <geometry>
+      <mesh filename="package://assembly_main_description/meshes/wheel_control_board_v7_2.stl" scale="0.001 0.001 0.001"/>
+    </geometry>
+    <material name="steel_satin"/>
+  </visual>
+  <collision>
+    <origin xyz="0.025 -0.0292 -0.0116" rpy="0 0 0"/>
+    <geometry>
+      <mesh filename="package://assembly_main_description/meshes/wheel_control_board_v7_2.stl" scale="0.001 0.001 0.001"/>
+    </geometry>
+  </collision>
+</link>
+<link name="raspi4_bracket_v3_1">
+  <inertial>
+    <origin xyz="0.0038877953241863647 -0.006733826728159031 0.009501909481815375" rpy="0 0 0"/>
+    <mass value="0.10147562490881655"/>
+    <inertia ixx="2.2e-05" iyy="3.2e-05" izz="3.7e-05" ixy="-9e-06" iyz="4e-06" ixz="-3e-06"/>
   </inertial>
   <visual>
     <origin xyz="0.04 -0.069282 -0.005" rpy="0 0 0"/>
     <geometry>
-      <mesh filename="package://assembly_main_description/meshes/raspi4_bracket_v1_1.stl" scale="0.001 0.001 0.001"/>
+      <mesh filename="package://assembly_main_description/meshes/raspi4_bracket_v3_1.stl" scale="0.001 0.001 0.001"/>
     </geometry>
     <material name="steel_satin"/>
@@ -59,5 +59,5 @@
     <origin xyz="0.04 -0.069282 -0.005" rpy="0 0 0"/>
     <geometry>
-      <mesh filename="package://assembly_main_description/meshes/raspi4_bracket_v1_1.stl" scale="0.001 0.001 0.001"/>
+      <mesh filename="package://assembly_main_description/meshes/raspi4_bracket_v3_1.stl" scale="0.001 0.001 0.001"/>
     </geometry>
   </collision>
@@ -83,34 +83,14 @@
   </collision>
 </link>
-<link name="lipo_bracket_v5_1">
-  <inertial>
-    <origin xyz="-0.007072287607066324 -0.03064999999999981 0.02557238675910756" rpy="0 0 0"/>
-    <mass value="0.15095338739595293"/>
-    <inertia ixx="0.000136" iyy="0.000109" izz="9.8e-05" ixy="-0.0" iyz="0.0" ixz="1e-06"/>
-  </inertial>
-  <visual>
-    <origin xyz="0.064425 -0.03065 -0.005" rpy="0 0 0"/>
-    <geometry>
-      <mesh filename="package://assembly_main_description/meshes/lipo_bracket_v5_1.stl" scale="0.001 0.001 0.001"/>
-    </geometry>
-    <material name="steel_satin"/>
-  </visual>
-  <collision>
-    <origin xyz="0.064425 -0.03065 -0.005" rpy="0 0 0"/>
-    <geometry>
-      <mesh filename="package://assembly_main_description/meshes/lipo_bracket_v5_1.stl" scale="0.001 0.001 0.001"/>
-    </geometry>
-  </collision>
-</link>
-<link name="DZ47B_63_circuit_breaker_holder_v3_1">
-  <inertial>
-    <origin xyz="0.03862239340692045 -0.022298666174134715 0.0029380076866297187" rpy="0 0 0"/>
-    <mass value="0.012274791356152887"/>
-    <inertia ixx="5e-06" iyy="1.5e-05" izz="2e-05" ixy="8e-06" iyz="0.0" ixz="-0.0"/>
+<link name="DZ47B_63_circuit_breaker_holder_v5_1">
+  <inertial>
+    <origin xyz="0.0378808179258513 -0.021870517177103727 0.0034323448804011907" rpy="0 0 0"/>
+    <mass value="0.018924792034229306"/>
+    <inertia ixx="8e-06" iyy="2.2e-05" izz="2.9e-05" ixy="1.2e-05" iyz="0.0" ixz="-0.0"/>
   </inertial>
   <visual>
     <origin xyz="0.076172 0.044934 -0.005" rpy="0 0 0"/>
     <geometry>
-      <mesh filename="package://assembly_main_description/meshes/DZ47B_63_circuit_breaker_holder_v3_1.stl" scale="0.001 0.001 0.001"/>
+      <mesh filename="package://assembly_main_description/meshes/DZ47B_63_circuit_breaker_holder_v5_1.stl" scale="0.001 0.001 0.001"/>
     </geometry>
     <material name="steel_satin"/>
@@ -119,189 +99,277 @@
     <origin xyz="0.076172 0.044934 -0.005" rpy="0 0 0"/>
     <geometry>
-      <mesh filename="package://assembly_main_description/meshes/DZ47B_63_circuit_breaker_holder_v3_1.stl" scale="0.001 0.001 0.001"/>
-    </geometry>
-  </collision>
-</link>
-<link name="arm_root_v4_1">
-  <inertial>
-    <origin xyz="0.02559296991432554 1.2574053551176077e-11 -0.009138901606431792" rpy="0 0 0"/>
-    <mass value="0.06457976620923557"/>
-    <inertia ixx="1.3e-05" iyy="2.4e-05" izz="1.9e-05" ixy="0.0" iyz="0.0" ixz="-1e-06"/>
-  </inertial>
-  <visual>
-    <origin xyz="-0.0615 -0.0 -0.045" rpy="0 0 0"/>
-    <geometry>
-      <mesh filename="package://assembly_main_description/meshes/arm_root_v4_1.stl" scale="0.001 0.001 0.001"/>
-    </geometry>
-    <material name="abs_white"/>
-  </visual>
-  <collision>
-    <origin xyz="-0.0615 -0.0 -0.045" rpy="0 0 0"/>
-    <geometry>
-      <mesh filename="package://assembly_main_description/meshes/arm_root_v4_1.stl" scale="0.001 0.001 0.001"/>
-    </geometry>
-  </collision>
-</link>
-<link name="pitch_1_test_v3_1">
-  <inertial>
-    <origin xyz="0.04097968346475826 0.0006820959366182021 -0.0001307207329616436" rpy="0 0 0"/>
-    <mass value="0.08186133563123103"/>
-    <inertia ixx="2.7e-05" iyy="4.3e-05" izz="3.7e-05" ixy="-1e-06" iyz="-0.0" ixz="-1e-05"/>
-  </inertial>
-  <visual>
-    <origin xyz="-0.1027 0.0 -0.05805" rpy="0 0 0"/>
-    <geometry>
-      <mesh filename="package://assembly_main_description/meshes/pitch_1_test_v3_1.stl" scale="0.001 0.001 0.001"/>
-    </geometry>
-    <material name="abs_white"/>
-  </visual>
-  <collision>
-    <origin xyz="-0.1027 0.0 -0.05805" rpy="0 0 0"/>
-    <geometry>
-      <mesh filename="package://assembly_main_description/meshes/pitch_1_test_v3_1.stl" scale="0.001 0.001 0.001"/>
-    </geometry>
-  </collision>
-</link>
-<link name="roll_1_test_v3_1">
-  <inertial>
-    <origin xyz="0.0363742814442784 0.0212000000095127 0.015160914691842164" rpy="0 0 0"/>
+      <mesh filename="package://assembly_main_description/meshes/DZ47B_63_circuit_breaker_holder_v5_1.stl" scale="0.001 0.001 0.001"/>
+    </geometry>
+  </collision>
+</link>
+<link name="wheel_control_board_v7_1">
+  <inertial>
+    <origin xyz="-0.01727366759971175 0.02421480381645276 0.006602625089643976" rpy="0 0 0"/>
+    <mass value="0.05597515361092653"/>
+    <inertia ixx="3.1e-05" iyy="1e-05" izz="4e-05" ixy="1e-06" iyz="-0.0" ixz="-0.0"/>
+  </inertial>
+  <visual>
+    <origin xyz="-0.0138 0.0292 -0.005" rpy="0 0 0"/>
+    <geometry>
+      <mesh filename="package://assembly_main_description/meshes/wheel_control_board_v7_1.stl" scale="0.001 0.001 0.001"/>
+    </geometry>
+    <material name="steel_satin"/>
+  </visual>
+  <collision>
+    <origin xyz="-0.0138 0.0292 -0.005" rpy="0 0 0"/>
+    <geometry>
+      <mesh filename="package://assembly_main_description/meshes/wheel_control_board_v7_1.stl" scale="0.001 0.001 0.001"/>
+    </geometry>
+  </collision>
+</link>
+<link name="lipo+battery_holder_v11_1">
+  <inertial>
+    <origin xyz="-0.014472410604743746 0.03065000000000157 0.01794464529626638" rpy="0 0 0"/>
+    <mass value="0.1619868833872407"/>
+    <inertia ixx="0.000116" iyy="0.000102" izz="0.00011" ixy="-0.0" iyz="0.0" ixz="0.0"/>
+  </inertial>
+  <visual>
+    <origin xyz="0.064425 0.03065 -0.005" rpy="0 0 0"/>
+    <geometry>
+      <mesh filename="package://assembly_main_description/meshes/lipo+battery_holder_v11_1.stl" scale="0.001 0.001 0.001"/>
+    </geometry>
+    <material name="steel_satin"/>
+  </visual>
+  <collision>
+    <origin xyz="0.064425 0.03065 -0.005" rpy="0 0 0"/>
+    <geometry>
+      <mesh filename="package://assembly_main_description/meshes/lipo+battery_holder_v11_1.stl" scale="0.001 0.001 0.001"/>
+    </geometry>
+  </collision>
+</link>
+<link name="arm_root_v6_1">
+  <inertial>
+    <origin xyz="0.028836205471188023 -6.461622099797368e-07 -0.0061030140912587336" rpy="0 0 0"/>
+    <mass value="0.05651259328313663"/>
+    <inertia ixx="1e-05" iyy="2.1e-05" izz="1.6e-05" ixy="-0.0" iyz="-0.0" ixz="-1e-06"/>
+  </inertial>
+  <visual>
+    <origin xyz="-0.0615 0.0 -0.044" rpy="0 0 0"/>
+    <geometry>
+      <mesh filename="package://assembly_main_description/meshes/arm_root_v6_1.stl" scale="0.001 0.001 0.001"/>
+    </geometry>
+    <material name="opaque254254255"/>
+  </visual>
+  <collision>
+    <origin xyz="-0.0615 0.0 -0.044" rpy="0 0 0"/>
+    <geometry>
+      <mesh filename="package://assembly_main_description/meshes/arm_root_v6_1.stl" scale="0.001 0.001 0.001"/>
+    </geometry>
+  </collision>
+</link>
+<link name="serial_servo_driver_board_x2_v3_1">
+  <inertial>
+    <origin xyz="0.01999999999999927 0.013999999418854537 -0.01849999999999563" rpy="0 0 0"/>
+    <mass value="0.4252482194783379"/>
+    <inertia ixx="9.8e-05" iyy="0.000117" izz="9.4e-05" ixy="-0.0" iyz="0.0" ixz="-0.0"/>
+  </inertial>
+  <visual>
+    <origin xyz="-0.0425 0.014 -0.103" rpy="0 0 0"/>
+    <geometry>
+      <mesh filename="package://assembly_main_description/meshes/serial_servo_driver_board_x2_v3_1.stl" scale="0.001 0.001 0.001"/>
+    </geometry>
+    <material name="steel_satin"/>
+  </visual>
+  <collision>
+    <origin xyz="-0.0425 0.014 -0.103" rpy="0 0 0"/>
+    <geometry>
+      <mesh filename="package://assembly_main_description/meshes/serial_servo_driver_board_x2_v3_1.stl" scale="0.001 0.001 0.001"/>
+    </geometry>
+  </collision>
+</link>
+<link name="arm_bracket_v14_1">
+  <inertial>
+    <origin xyz="-0.005004825728865167 0.009999999984475738 0.04726352833341586" rpy="0 0 0"/>
+    <mass value="0.21684183891762862"/>
+    <inertia ixx="0.000236" iyy="0.000211" izz="7e-05" ixy="-0.0" iyz="0.0" ixz="3.5e-05"/>
+  </inertial>
+  <visual>
+    <origin xyz="-0.047 0.01 -0.005" rpy="0 0 0"/>
+    <geometry>
+      <mesh filename="package://assembly_main_description/meshes/arm_bracket_v14_1.stl" scale="0.001 0.001 0.001"/>
+    </geometry>
+    <material name="steel_satin"/>
+  </visual>
+  <collision>
+    <origin xyz="-0.047 0.01 -0.005" rpy="0 0 0"/>
+    <geometry>
+      <mesh filename="package://assembly_main_description/meshes/arm_bracket_v14_1.stl" scale="0.001 0.001 0.001"/>
+    </geometry>
+  </collision>
+</link>
+<link name="roll_1_test_v5_1">
+  <inertial>
+    <origin xyz="0.036374051351653836 0.021199665031561798 0.015160509124310162" rpy="0 0 0"/>
     <mass value="0.07353297901744495"/>
     <inertia ixx="2.4e-05" iyy="2.9e-05" izz="2.1e-05" ixy="0.0" iyz="-0.0" ixz="-1e-06"/>
   </inertial>
   <visual>
-    <origin xyz="-0.1649 0.02035 -0.0635" rpy="0 0 0"/>
-    <geometry>
-      <mesh filename="package://assembly_main_description/meshes/roll_1_test_v3_1.stl" scale="0.001 0.001 0.001"/>
+    <origin xyz="-0.167022 0.02086 -0.07071" rpy="0 0 0"/>
+    <geometry>
+      <mesh filename="package://assembly_main_description/meshes/roll_1_test_v5_1.stl" scale="0.001 0.001 0.001"/>
+    </geometry>
+    <material name="oak"/>
+  </visual>
+  <collision>
+    <origin xyz="-0.167022 0.02086 -0.07071" rpy="0 0 0"/>
+    <geometry>
+      <mesh filename="package://assembly_main_description/meshes/roll_1_test_v5_1.stl" scale="0.001 0.001 0.001"/>
+    </geometry>
+  </collision>
+</link>
+<link name="pitch_2_test_v8_1">
+  <inertial>
+    <origin xyz="0.03178013194406809 0.0006984560339173065 2.2244498183721095e-07" rpy="0 0 0"/>
+    <mass value="0.058119652228533734"/>
+    <inertia ixx="1e-05" iyy="1.7e-05" izz="2.2e-05" ixy="-1e-06" iyz="0.0" ixz="0.0"/>
+  </inertial>
+  <visual>
+    <origin xyz="-0.223422 -0.00034 -0.07071" rpy="0 0 0"/>
+    <geometry>
+      <mesh filename="package://assembly_main_description/meshes/pitch_2_test_v8_1.stl" scale="0.001 0.001 0.001"/>
     </geometry>
     <material name="abs_white"/>
   </visual>
   <collision>
-    <origin xyz="-0.1649 0.02035 -0.0635" rpy="0 0 0"/>
-    <geometry>
-      <mesh filename="package://assembly_main_description/meshes/roll_1_test_v3_1.stl" scale="0.001 0.001 0.001"/>
-    </geometry>
-  </collision>
-</link>
-<link name="pitch_2_test_v3_1">
-  <inertial>
-    <origin xyz="0.029877529047602214 0.0001958957866964999 -2.9469195139686377e-10" rpy="0 0 0"/>
-    <mass value="0.06668343069893205"/>
-    <inertia ixx="1.4e-05" iyy="2e-05" izz="2.6e-05" ixy="-1e-06" iyz="-0.0" ixz="-0.0"/>
-  </inertial>
-  <visual>
-    <origin xyz="-0.2213 -0.00085 -0.0635" rpy="0 0 0"/>
-    <geometry>
-      <mesh filename="package://assembly_main_description/meshes/pitch_2_test_v3_1.stl" scale="0.001 0.001 0.001"/>
-    </geometry>
-    <material name="abs_white"/>
-  </visual>
-  <collision>
-    <origin xyz="-0.2213 -0.00085 -0.0635" rpy="0 0 0"/>
-    <geometry>
-      <mesh filename="package://assembly_main_description/meshes/pitch_2_test_v3_1.stl" scale="0.001 0.001 0.001"/>
-    </geometry>
-  </collision>
-</link>
-<link name="roll_2_test_v3_1">
-  <inertial>
-    <origin xyz="0.036375491747628774 0.021200000009496393 0.015187663571532395" rpy="0 0 0"/>
+    <origin xyz="-0.223422 -0.00034 -0.07071" rpy="0 0 0"/>
+    <geometry>
+      <mesh filename="package://assembly_main_description/meshes/pitch_2_test_v8_1.stl" scale="0.001 0.001 0.001"/>
+    </geometry>
+  </collision>
+</link>
+<link name="roll_2_test_v5_1">
+  <inertial>
+    <origin xyz="0.036375261655003766 0.021199665031546605 0.015187258004001114" rpy="0 0 0"/>
     <mass value="0.07365581710871624"/>
     <inertia ixx="2.4e-05" iyy="2.9e-05" izz="2.1e-05" ixy="0.0" iyz="-0.0" ixz="-1e-06"/>
   </inertial>
   <visual>
-    <origin xyz="-0.2675 0.02015 -0.0635" rpy="0 0 0"/>
-    <geometry>
-      <mesh filename="package://assembly_main_description/meshes/roll_2_test_v3_1.stl" scale="0.001 0.001 0.001"/>
-    </geometry>
-    <material name="abs_white"/>
-  </visual>
-  <collision>
-    <origin xyz="-0.2675 0.02015 -0.0635" rpy="0 0 0"/>
-    <geometry>
-      <mesh filename="package://assembly_main_description/meshes/roll_2_test_v3_1.stl" scale="0.001 0.001 0.001"/>
-    </geometry>
-  </collision>
-</link>
-<link name="hand_unit_v3_1">
-  <inertial>
-    <origin xyz="0.031683675390487276 -0.00023986066792197516 -0.011102966860764112" rpy="0 0 0"/>
-    <mass value="0.0952280970557457"/>
-    <inertia ixx="4.8e-05" iyy="7.4e-05" izz="5.4e-05" ixy="-0.0" iyz="1e-06" ixz="1.9e-05"/>
-  </inertial>
-  <visual>
-    <origin xyz="-0.3239 -0.00105 -0.0635" rpy="0 0 0"/>
-    <geometry>
-      <mesh filename="package://assembly_main_description/meshes/hand_unit_v3_1.stl" scale="0.001 0.001 0.001"/>
-    </geometry>
-    <material name="abs_white"/>
-  </visual>
-  <collision>
-    <origin xyz="-0.3239 -0.00105 -0.0635" rpy="0 0 0"/>
-    <geometry>
-      <mesh filename="package://assembly_main_description/meshes/hand_unit_v3_1.stl" scale="0.001 0.001 0.001"/>
-    </geometry>
-  </collision>
-</link>
-<link name="hand_finger_v7_1">
-  <inertial>
-    <origin xyz="0.03630500457367125 0.02170000000000132 0.024617294394885247" rpy="0 0 0"/>
-    <mass value="0.024732672038933038"/>
-    <inertia ixx="7e-06" iyy="1.5e-05" izz="1.8e-05" ixy="-0.0" iyz="0.0" ixz="-4e-06"/>
-  </inertial>
-  <visual>
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
File: urdf/komarm.urdf (robot description, URDF)
Before this commit: robot assembly_main, 13 links, 12 joints
Links:
- removed link DZ47B_63_circuit_breaker_holder_v3_1
- removed link arm_bracket_temp_v12_1
- removed link arm_root_v4_1
- removed link hand_finger_v7_1
- removed link hand_unit_v3_1
- removed link lipo_bracket_v5_1
- removed link pitch_1_test_v3_1
- removed link pitch_2_test_v3_1
- removed link raspi4_bracket_v1_1
- removed link roll_1_test_v3_1
- removed link roll_2_test_v3_1
- added link DZ47B_63_circuit_breaker_holder_v5_1, mass 0.018924792034229306; collision mesh filename=../meshes/DZ47B_63_circuit_breaker_holder_v5_1.stl scale=0.001 0.001 0.001; visual mesh filename=../meshes/DZ47B_63_circuit_breaker_holder_v5_1.stl scale=0.001 0.001 0.001
- added link arm_bracket_v14_1, mass 0.21684183891762862; collision mesh filename=../meshes/arm_bracket_v14_1.stl scale=0.001 0.001 0.001; visual mesh filename=../meshes/arm_bracket_v14_1.stl scale=0.001 0.001 0.001
- added link arm_root_v6_1, mass 0.05651259328313663; collision mesh filename=../meshes/arm_root_v6_1.stl scale=0.001 0.001 0.001; visual mesh filename=../meshes/arm_root_v6_1.stl scale=0.001 0.001 0.001
- added link hand_finger_v38_1, mass 0.07994136386082434; collision mesh filename=../meshes/hand_finger_v38_1.stl scale=0.001 0.001 0.001; visual mesh filename=../meshes/hand_finger_v38_1.stl scale=0.001 0.001 0.001
- added link hand_unit_v24_1, mass 0.13230659416117943; collision mesh filename=../meshes/hand_unit_v24_1.stl scale=0.001 0.001 0.001; visual mesh filename=../meshes/hand_unit_v24_1.stl scale=0.001 0.001 0.001
- added link lipo+battery_holder_v11_1, mass 0.1619868833872407; collision mesh filename=../meshes/lipo+battery_holder_v11_1.stl scale=0.001 0.001 0.001; visual mesh filename=../meshes/lipo+battery_holder_v11_1.stl scale=0.001 0.001 0.001
- added link pitch_1_test_v10_1, mass 0.11843544806781975; collision mesh filename=../meshes/pitch_1_test_v10_1.stl scale=0.001 0.001 0.001; visual mesh filename=../meshes/pitch_1_test_v10_1.stl scale=0.001 0.001 0.001
- added link pitch_2_test_v8_1, mass 0.058119652228533734; collision mesh filename=../meshes/pitch_2_test_v8_1.stl scale=0.001 0.001 0.001; visual mesh filename=../meshes/pitch_2_test_v8_1.stl scale=0.001 0.001 0.001
- added link raspi4_bracket_v3_1, mass 0.10147562490881655; collision mesh filename=../meshes/raspi4_bracket_v3_1.stl scale=0.001 0.001 0.001; visual mesh filename=../meshes/raspi4_bracket_v3_1.stl scale=0.001 0.001 0.001
- added link roll_1_test_v5_1, mass 0.07353297901744495; collision mesh filename=../meshes/roll_1_test_v5_1.stl scale=0.001 0.001 0.001; visual mesh filename=../meshes/roll_1_test_v5_1.stl scale=0.001 0.001 0.001
- added link roll_2_test_v5_1, mass 0.07365581710871624; collision mesh filename=../meshes/roll_2_test_v5_1.stl scale=0.001 0.001 0.001; visual mesh filename=../meshes/roll_2_test_v5_1.stl scale=0.001 0.001 0.001
- added link serial_servo_driver_board_x2_v3_1, mass 0.4252482194783379; collision mesh filename=../meshes/serial_servo_driver_board_x2_v3_1.stl scale=0.001 0.001 0.001; visual mesh filename=../meshes/serial_servo_driver_board_x2_v3_1.stl scale=0.001 0.001 0.001
- added link wheel_control_board_v7_1, mass 0.05597515361092653; collision mesh filename=../meshes/wheel_control_board_v7_1.stl scale=0.001 0.001 0.001; visual mesh filename=../meshes/wheel_control_board_v7_1.stl scale=0.001 0.001 0.001
- added link wheel_control_board_v7_2, mass 0.05597515361092653; collision mesh filename=../meshes/wheel_control_board_v7_2.stl scale=0.001 0.001 0.001; visual mesh filename=../meshes/wheel_control_board_v7_2.stl scale=0.001 0.001 0.001
- link base_link: mass 10.00 -> 4.27590428722208
Joints:
- removed joint Revolute_6
- removed joint Rigid 16
- removed joint Rigid 26
- removed joint Rigid 4
- added joint Rigid 27: type fixed, parent base_link, child wheel_control_board_v7_1, origin xyz=0.0138 -0.0292 0.005 rpy=0 0 0
- added joint Rigid 31: type fixed, parent base_link, child lipo+battery_holder_v11_1, origin xyz=-0.064425 -0.03065 0.005 rpy=0 0 0
- added joint Rigid 45: type fixed, parent arm_bracket_v14_1, child arm_root_v6_1, origin xyz=0.0145 0.01 0.039 rpy=0 0 0
- added joint Rigid 46: type fixed, parent arm_bracket_v14_1, child serial_servo_driver_board_x2_v3_1, origin xyz=-0.0045 -0.004 0.098 rpy=0 0 0
- added joint Rigid 47: type fixed, parent base_link, child arm_bracket_v14_1, origin xyz=0.047 -0.01 0.005 rpy=0 0 0
- added joint Rigid 6: type fixed, parent wheel_control_board_v7_1, child wheel_control_board_v7_2, origin xyz=-0.0388 0.0584 0.0066 rpy=0 0 0
- joint Revolute_1: axis 0.0 -0.0 -1.0 -> -0.0 0.0 1.0; child pitch_1_test_v3_1 -> pitch_1_test_v10_1; limit lower=-1.570796 upper=1.570796 effort=1.5 velocity=4.0 -> effort=1.5 velocity=4.0; origin xyz=0.0412 -0.0 0.01305 rpy=0 0 0 -> xyz=0.0424 0.0 0.0118 rpy=0 0 0; parent arm_root_v4_1 -> arm_root_v6_1; type revolute -> continuous
- joint Revolute_2: child roll_1_test_v3_1 -> roll_1_test_v5_1; origin xyz=0.0622 -0.02035 0.00545 rpy=0 0 0 -> xyz=0.063122 -0.02086 0.01491 rpy=0 0 0; parent pitch_1_test_v3_1 -> pitch_1_test_v10_1
- joint Revolute_3: axis 1.0 0.0 0.0 -> -1.0 0.0 -0.0; child pitch_2_test_v3_1 -> pitch_2_test_v8_1; parent roll_1_test_v3_1 -> roll_1_test_v5_1
- joint Revolute_4: child roll_2_test_v3_1 -> roll_2_test_v5_1; origin xyz=0.0462 -0.021 0.0 rpy=0 0 0 -> xyz=0.0462 -0.0208 0.0 rpy=0 0 0; parent pitch_2_test_v3_1 -> pitch_2_test_v8_1
- joint Revolute_5: child hand_unit_v3_1 -> hand_unit_v24_1; parent roll_2_test_v3_1 -> roll_2_test_v5_1
- joint Rigid 17: child DZ47B_63_circuit_breaker_holder_v3_1 -> DZ47B_63_circuit_breaker_holder_v5_1
- joint Rigid 7: child raspi4_bracket_v1_1 -> raspi4_bracket_v3_1
- joint Rigid 8: parent raspi4_bracket_v1_1 -> raspi4_bracket_v3_1
